File: hw/Keyboard-Right.kicad_sch (KiCad schematic)
At the start: 17 parts, among them P1000 Current-Probe, X1000 Mounting-Hole-M3, X1001 Mounting-Hole-M3, X1002 Mounting-Hole-M3, X1003 Mounting-Hole-M3, X1004 Distance-Bolt_M3x5, X1005 Distance-Bolt_M3x5, X1006 Distance-Bolt_M3x5, X1007 Distance-Bolt_M3x5, X1008 Screw M3x10, X1009 Screw M3x10, X1010 Screw M3x10, X1011 Screw M3x10, X1012 Screw M3x10, X1013 Screw M3x10, X1014 Screw M3x10, X1015 Screw M3x10

Commit message: Update schematic:
- Add ESD protection.
- Adjust distance bolts so they fit to the MX mounting plate.
- Make key layout symmetric.
- Add resistor to TX driver outputs.
- Use alternate IO functions on inter-board connectors.
Parts:
- X1004, X1005, X1006, X1007: footprint Keyboard:DistanceBolt-M3x5 -> Keyboard:DistanceBolt-6x3.5; symbol Keyboard:Distance-Bolt_M3x5 -> Keyboard:Distance-Bolt_6x3.5
Changed lines of the file:
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@@
     (pin "1")
   )
-  (symbol (lib_id "Keyboard:Distance-Bolt_M3x5") (at 27.94 78.74 0) (unit 1)
+  (symbol (lib_id "Keyboard:Distance-Bolt_6x3.5") (at 27.94 78.74 0) (unit 1)
     (in_bom yes) (on_board yes) (fields_autoplaced)
     (property "Reference" "X1007" (id 0) (at 31.115 77.8315 0)
@@
       (effects (font (size 1.27 1.27)) (justify left))
     )
-    (property "Footprint" "Keyboard:DistanceBolt-M3x5" (id 2) (at 27.94 78.74 0)
+    (property "Footprint" "Keyboard:DistanceBolt-6x3.5" (id 2) (at 27.94 78.74 0)
       (effects (font (size 1.27 1.27)) hide)
     )
@@
     )
   )
-  (symbol (lib_id "Keyboard:Distance-Bolt_M3x5") (at 27.94 66.04 0) (unit 1)
+  (symbol (lib_id "Keyboard:Distance-Bolt_6x3.5") (at 27.94 66.04 0) (unit 1)
     (in_bom yes) (on_board yes) (fields_autoplaced)
     (property "Reference" "X1005" (id 0) (at 31.115 65.1315 0)
@@
       (effects (font (size 1.27 1.27)) (justify left))
     )
-    (property "Footprint" "Keyboard:DistanceBolt-M3x5" (id 2) (at 27.94 66.04 0)
+    (property "Footprint" "Keyboard:DistanceBolt-6x3.5" (id 2) (at 27.94 66.04 0)
       (effects (font (size 1.27 1.27)) hide)
     )
@@
     )
   )
-  (symbol (lib_id "Keyboard:Distance-Bolt_M3x5") (at 27.94 72.39 0) (unit 1)
+  (symbol (lib_id "Keyboard:Distance-Bolt_6x3.5") (at 27.94 72.39 0) (unit 1)
     (in_bom yes) (on_board yes) (fields_autoplaced)
     (property "Reference" "X1006" (id 0) (at 31.115 71.4815 0)
@@
       (effects (font (size 1.27 1.27)) (justify left))
     )
-    (property "Footprint" "Keyboard:DistanceBolt-M3x5" (id 2) (at 27.94 72.39 0)
+    (property "Footprint" "Keyboard:DistanceBolt-6x3.5" (id 2) (at 27.94 72.39 0)
       (effects (font (size 1.27 1.27)) hide)
     )
@@
     )
   )
-  (symbol (lib_id "Keyboard:Distance-Bolt_M3x5") (at 27.94 59.69 0) (unit 1)
+  (symbol (lib_id "Keyboard:Distance-Bolt_6x3.5") (at 27.94 59.69 0) (unit 1)
     (in_bom yes) (on_board yes) (fields_autoplaced)
     (property "Reference" "X1004" (id 0) (at 31.115 58.7815 0)
@@
       (effects (font (size 1.27 1.27)) (justify left))
     )
-    (property "Footprint" "Keyboard:DistanceBolt-M3x5" (id 2) (at 27.94 59.69 0)
+    (property "Footprint" "Keyboard:DistanceBolt-6x3.5" (id 2) (at 27.94 59.69 0)
       (effects (font (size 1.27 1.27)) hide)
     )
